File: hardware/generic_maxi_1/generic_maxi_1.sch (EAGLE design)
At the start: 17 parts, among them IC1 MEGA48/88/168-PU, IC2 RFM12, Q1 4MHz

Commit message: use .org domain
Other:
- note added: "Copyright (c) Uwe Freese, www.smarthomatic.org"
- note removed: "Copyright (c) Uwe Freese, www.smarthomatic.com"
Changed lines of the file:
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@@
 <text x="121.92" y="-45.72" size="2.1844" layer="97">Date: 02.12.2012</text>
 <text x="66.04" y="-45.72" size="2.1844" layer="97">Rev 1.0</text>
-<text x="66.04" y="-50.8" size="2.1844" layer="97">Copyright (c) Uwe Freese, www.smarthomatic.com</text>
+<text x="66.04" y="-50.8" size="2.1844" layer="97">Copyright (c) Uwe Freese, www.smarthomatic.org</text>
 </plain>
 <instances>
