File: hardware/generic_micro_1/generic_micro_1.sch (EAGLE design)
At the start: 23 parts, among them IC1 MEGA48/88/168-AU, IC2 RFM12, IC3 LP2950Z

Commit message: use .org domain
Other:
- note added: "Copyright (c) Uwe Freese, www.smarthomatic.org"
- note removed: "Copyright (c) Uwe Freese, www.smarthomatic.com"
Changed lines of the file:
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@@
 <text x="116.84" y="-48.26" size="2.1844" layer="97">Date: 08.12.2012</text>
 <text x="66.04" y="-48.26" size="2.1844" layer="97">Rev 1.0</text>
-<text x="66.04" y="-53.34" size="2.1844" layer="97">Copyright (c) Uwe Freese, www.smarthomatic.com</text>
+<text x="66.04" y="-53.34" size="2.1844" layer="97">Copyright (c) Uwe Freese, www.smarthomatic.org</text>
 </plain>
 <instances>
