File: hardware/generic_midi_1/generic_midi_1.brd (EAGLE design)
At the start: 47.3 x 44.8 mm, 20 parts, among them IC1 MEGA168/328, IC2 RFM12

Commit message: Correct label of PD1/TX pin.
Parts:
- JP8: value PD5 -> PD1/TX
Changed lines of the file:
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@@
 <layer number="23" name="tOrigins" color="15" fill="1" visible="no" active="yes"/>
 <layer number="24" name="bOrigins" color="15" fill="1" visible="no" active="yes"/>
-<layer number="25" name="tNames" color="7" fill="1" visible="no" active="yes"/>
-<layer number="26" name="bNames" color="7" fill="1" visible="no" active="yes"/>
-<layer number="27" name="tValues" color="7" fill="1" visible="no" active="yes"/>
-<layer number="28" name="bValues" color="7" fill="1" visible="no" active="yes"/>
+<layer number="25" name="tNames" color="7" fill="1" visible="yes" active="yes"/>
+<layer number="26" name="bNames" color="7" fill="1" visible="yes" active="yes"/>
+<layer number="27" name="tValues" color="7" fill="1" visible="yes" active="yes"/>
+<layer number="28" name="bValues" color="7" fill="1" visible="yes" active="yes"/>
 <layer number="29" name="tStop" color="7" fill="3" visible="no" active="yes"/>
 <layer number="30" name="bStop" color="7" fill="6" visible="no" active="yes"/>
@@
 <attribute name="VALUE" x="8.1915" y="31.1912" size="1.27" layer="27" ratio="10"/>
 </element>
-<element name="JP8" library="pinhead" package="1X01" value="PD5" x="13.335" y="19.3675" smashed="yes">
-<attribute name="VALUE" x="11.7475" y="18.0975" size="1.27" layer="27" rot="R90"/>
+<element name="JP8" library="pinhead" package="1X01" value="PD1/TX" x="13.335" y="19.3675" smashed="yes">
+<attribute name="VALUE" x="12.065" y="20.0025" size="1.27" layer="27" rot="R180"/>
 </element>
 </elements>
