File: hardware/rgb_dimmer_1/rgb_dimmer_1.brd (EAGLE design)
At the start: 47.3 x 44.1 mm, 23 parts, among them IC1 MEGA168/328, IC2 RFM12, IC3 LP2950Z, T1 BC337, T2 BC337, T3 BC337

Commit message: update RGB dimmer PCB
Parts:
- added C2: 100µ, rcl:E2,5-6
- moved JP2 4.14 mm to (3.49, 24.3)
- moved JP6 3.19 mm to (3.49, 30.5)
- moved R8 2.54 mm to (10.8, 33.0)
- moved T3 0.63 mm to (17.5, 31.4)
Connections:
- net +5V: now also C2.+
- net GND: now also C2.-
Routing:
- net N$8: track 46.0 -> 39.2 mm, vias 0 -> 2
- net GND: track 151.5 -> 156.0 mm
- net +5V: track 54.9 -> 58.4 mm
- net N$1: track 3.49 -> 5.85 mm
- net N$19: track 5.08 -> 3.18 mm
- net N$18: track 3.57 -> 2.22 mm
- net N$16: track 3.81 -> 3.00 mm
- net N$10: track 28.3 -> 27.6 mm
Other:
- board text added: "Rev 1.1"
- board text removed: "Rev 1.0"
