File: hardware/power_switch_1/power_switch_1.brd (EAGLE design)
At the start: 50 x 50 mm, 21 parts, among them IC1 MEGA168/328, IC2 RFM12, IC3 LP2950Z, K1 FTR-K1C, T1 BC547, X1 SW Out

Commit message: In PCB V1.1, the power pin of the RFM module is connected to an ATMega pin to allow restart if needed.
Parts:
- added C2: 1µ, capacitor-wima:C5B3.5
Connections:
- new net N$22: C2.1, IC1.26, IC2.3, IC2.9
- net +3V3: no longer IC2.3, IC2.9
- net GND: now also C2.2
Routing:
- net N$22: track 0.00 -> 56.0 mm, vias 0 -> 3
- net +3V3: track 94.2 -> 79.2 mm
- net GND: track 114.2 -> 115.5 mm
- net N$4: track 41.0 -> 41.8 mm
Other:
- board text added: "Rev 1.1"
- board text removed: "D:/Eigene Dateien/smarthomatic/logo/logo_black 150x133.bmp"
- board text removed: "Rev 1.0"
