File: hardware/shutter_control/shutter_control.brd (EAGLE design)
At the start: 50 x 50 mm, 32 parts, among them IC1 MEGA168/328, IC2 RFM12, IC3 LP2950Z, K1 G6D-1A-ASI5VDC, K2 G6D-1A-ASI5VDC, T1 BC547, T2 BC547, T3 BC547, X1 SW Out

Commit message: First version of shutter control schematics and PCB layout.
Parts:
- C1: value 10Âµ -> 10µ
- C2: value 1Âµ -> 1µ
Changed lines of the file:
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@@
 <attribute name="VALUE" x="47.3837" y="37.211" size="1.27" layer="27" ratio="10" rot="R270"/>
 </element>
-<element name="C1" library="rcl" package="E1,8-4" value="10Âµ" x="32.385" y="45.085" smashed="yes" rot="R180">
+<element name="C1" library="rcl" package="E1,8-4" value="10µ" x="32.385" y="45.085" smashed="yes" rot="R180">
 <attribute name="NAME" x="36.2585" y="44.0055" size="1.27" layer="25" ratio="10" rot="R180"/>
 <attribute name="VALUE" x="34.3535" y="42.7355" size="1.27" layer="27" ratio="10" rot="R180"/>
@@
 <attribute name="NAME" x="17.1196" y="3.175" size="1.778" layer="25" ratio="10" rot="R180"/>
 </element>
-<element name="C2" library="capacitor-wima" package="C5B3.5" value="1Âµ" x="11.43" y="26.67" smashed="yes" rot="R180">
+<element name="C2" library="capacitor-wima" package="C5B3.5" value="1µ" x="11.43" y="26.67" smashed="yes" rot="R180">
 <attribute name="NAME" x="11.43" y="28.702" size="1.27" layer="25" ratio="10"/>
 <attribute name="VALUE" x="10.16" y="29.972" size="1.27" layer="27" ratio="10" rot="R180"/>
